Commit message: copy of customized lio-sam for rm 2024. Feature: livox customized pointcloud, better support for mid 360, potential integration with encoder velocity

File: config/robot.urdf.xacro (robot description, xacro)
@@ -1,35 +1,12 @@
-<?xml version="1.0"?>
-<robot name="lio" xmlns:xacro="http://tixiaoshan.github.io/">
-  <xacro:property name="PI" value="3.1415926535897931" />
-  <link name="chassis_link"></link>
-  <link name="base_link"></link>
-  <joint name="base_link_joint" type="fixed">
-    <parent link="base_link"/>
-    <child link="chassis_link" />
-    <origin xyz="0 0 0" rpy="0 0 0" />
-  </joint>
-  <link name="lidar_link"> </link>
-  <joint name="lidar_joint" type="fixed">
-    <parent link="base_link" />
-    <child link="lidar_link" />
-    <origin xyz="0 0 0" rpy="0 0 0" />
-  </joint>
-  <link name="imu_link"> </link>
-  <joint name="imu_joint" type="fixed">
-    <parent link="chassis_link" />
-    <child link="imu_link" />
-    <origin xyz="0 0 0" rpy="0 0 0" />
-  </joint>
-  <link name="laser_sensor_frame"> </link>
-  <joint name="laser_joint" type="fixed">
-    <parent link="imu_link" />
-    <child link="laser_sensor_frame" />
-    <origin xyz="0 0 0" rpy="0 0 0" />
-  </joint>
-  <link name="navsat_link"> </link>
-  <joint name="navsat_joint" type="fixed">
-    <parent link="chassis_link" />
-    <child link="navsat_link" />
-    <origin xyz="0 0 0" rpy="0 0 0" />
+<?xml version="1.0" encoding="utf-8"?>
+<robot name="sentry"
+  xmlns:xacro="http://ros.org/wiki/xacro">
+  <link name="livox_frame" />
+  <link name = "base_link_slam" />
+  <joint name="base_joint" type="fixed">
+    <origin xyz="-0.105 0.0 -0.460" rpy="0.0 0.0 0.0" />
+    <parent link="livox_frame" />
+    <child link="base_link_slam" />
+    <axis xyz= "0 1 0" />
   </joint>
 </robot>

Commit message: update urdf

File: config/robot.urdf.xacro (robot description, xacro)
@@ -5,5 +5,5 @@
   <link name = "base_link_slam" />
   <joint name="base_joint" type="fixed">
-    <origin xyz="-0.105 0.0 -0.460" rpy="0.0 0.0 0.0" />
+    <origin xyz="0.0 0.0 -0.460" rpy="0.0 0.0 0.0" />
     <parent link="livox_frame" />
     <child link="base_link_slam" />
